File: Z80.kicad_pcb (KiCad board)
At the start: 2 copper layers, 85.1 x 111.8 mm, 38 parts, among them J1 USB_B, J2 Conn_01x16_Male, J3 Conn_01x08_Male, U1 74HCT04, U2 68B50, U3 Z80CPU, U4 2764, U5 628128, U6 74LS32, U7 CH340G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

Commit message: Send to github
Routing:
- net GND: vias 20 -> 21
Changed lines of the file:
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@@
-(kicad_pcb (version 20171130) (host pcbnew "(5.0.0-rc2-dev-493-gd776eaca8)")
+(kicad_pcb (version 20171130) (host pcbnew "(5.0.0)")
   (general
     (thickness 1.6)
     (drawings 45)
-    (tracks 1240)
+    (tracks 1241)
     (zones 0)
     (modules 38)
@@
       (hpglpennumber 1)
       (hpglpenspeed 20)
-      (hpglpendiameter 15)
+      (hpglpendiameter 15.000000)
       (psnegative false)
       (psa4output false)
@@
       (drillshape 0)
       (scaleselection 1)
-      (outputdirectory gerber/))
+      (outputdirectory "gerber/"))
   )
   (net 0 "")
@@
   (segment (start 148.59 76.2) (end 151.17 76.2) (width 0.25) (layer B.Cu) (net 13))
   (via (at 106.68 63.5) (size 0.8) (drill 0.4) (layers F.Cu B.Cu) (net 13))
+  (via (at 157.9245 108.1405) (size 0.8) (drill 0.4) (layers F.Cu B.Cu) (net 13))
   (segment (start 92.71 136.525) (end 92.71 135.3997) (width 0.25) (layer B.Cu) (net 14))
   (segment (start 92.71 135.3997) (end 93.0733 135.3997) (width 0.25) (layer B.Cu) (net 14))
