File: Z80.sch (KiCad schematic (older format))
At the start: 36 parts, among them J1 USB_B, J2 Conn_01x16_Male, J3 Conn_01x08_Male, J4 Conn_01x02_Male, SW1 SW_Push_Dual, U1 74HCT04, U2 68B50, U3 Z80CPU, U4 2764, U5 628128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

Commit message: Added schematic plots
Connections:
- wire segments 187 -> 196
Other:
- note added: "Aidan Lawrence\nwww.aidanlawrence.com\nAdapted from Grant Searle\nsearle.hostei.com"
- note added: "COM & Serial"
- note added: "I/O Headers"
- note added: "LED bars"
- note added: "RAM & ROM"
- note added: "System Clock"
- note added: "Z80 CPU"
- moved on the sheet: U4
